Commit message: Remove main.py, spacemouse_ball.py, robot_modified.urdf, and robot_simplified.urdf. Update README.md to reflect the new gripper drill attachment and changes in the robot's URDF structure. Modify simulate_robot.py to use the new gripper drill URDF and adjust end effector identification logic.

File: robot_pybullet.urdf (robot description, URDF)
Before this commit: robot owl_robot, 10 links, 9 joints
Links:
- added link camera_frame, mass 1e-9
- added link gripper_drill_combined_v1, mass 0.20782; collision mesh filename=/Users/keval/Documents/VSCode/owl-spacemouse-controller/owl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; visual mesh filename=/Users/keval/Documents/VSCode/owl-spacemouse-controller/owl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
- added link target_frame, mass 1e-9
Joints:
- added joint gripper_to_target: type fixed, parent gripper_drill_combined_v1, child target_frame, origin xyz=0.034827 0.094877 0.146175 rpy=0 0 0, axis 0 0 0
- added joint robot_gripper_base_joint: type fixed, parent tcp, child gripper_drill_combined_v1, origin xyz=0.0 0.0 -0.017 rpy=0 0 3.14
- added joint target_to_camera: type fixed, parent target_frame, child camera_frame, origin xyz=-0.106874 -0.094877 -0.105064 rpy=0 -1.5708 0, axis 0 0 0
- joint virtual_joint: origin xyz=0 -0.6 0.07 rpy=0 0 3.14 -> xyz=0 0 0 rpy=0 0 0
